File: Diseño/modulargas.kicad_pcb (KiCad board)
At the start: 2 copper layers, 100 x 150 mm, 53 parts, among them J1 MiSD, J10 DLUZ, J11 DISPLAY, J13 RJ45_Shielded, J2 GPS, J3 DS3231, J4 ITG, J5 TECLADO, J7 IMPRESORA, J8 PONTENCIA, J9 Conn_01x02_Socket, K1 Fujitsu_FTR-LYCA005x, K2 Fujitsu_FTR-LYCA005x, Q1 BC548, Q2 BC548, Q3 BC548, Q4 BC548, U2 MAX232, U3 Pico, U4 NODEMCU-32S

Commit message: Actualization
Se terminaron de hacer las conexiones
Parts:
- removed the G*** at (97.8, 62.0)
- added G***: LOGO, LOGO, B.Cu at (100.1, 73.4)
- added G***: LOGO, LOGO, B.Cu at (101.0, 89.0)
- moved BT2 0.65 mm to (111.8, 111.3)
- renumbered SD3 to CARGADOR, J11 to DISPLAY, J10 to DLUZ, J2 to GPS, J7 to IMPRESORA, J4 to MPU/ACE, J1 to MiSD, J8 to POTENCIA, J13 to RJ45, J3 to RTC, SD2 to StepDown, SD1 to StepUp, J5 to TECLADO
Routing:
- net /r4: track 70.5 -> 114.8 mm
- net +12V: track 57.6 -> 75.1 mm
- net GND: track 0.00 -> 9.73 mm, vias 0 -> 1
- net +5V: track 308.2 -> 314.1 mm
